Commit message: bicycle + manipulator properly imported in Rviz

File: my_workspace/src/ros2_control_demos/example_11/description/urdf/carlikebot.urdf.xacro (robot description, xacro)
@@ -1,13 +1,18 @@
 <?xml version="1.0"?>
-<!-- 4 Wheel Robot with front steering and rear drive -->
 <robot xmlns:xacro="http://www.ros.org/wiki/xacro" name="carlikebot_robot">
-  <xacro:arg name="prefix" default="" />
+  <xacro:arg name="prefix" default="car_" />
   <xacro:include filename="$(find ros2_control_demo_description)/carlikebot/urdf/carlikebot_description.urdf.xacro" />
-  <!-- Import Rviz colors -->
+  <xacro:include filename="$(find ros2_control_demo_description)/r6bot/urdf/r6bot_description.urdf.xacro" />
   <xacro:include filename="$(find ros2_control_demo_description)/carlikebot/urdf/carlikebot.materials.xacro" />
-  <!-- Import carlikebot ros2_control description -->
   <xacro:include filename="$(find ros2_control_demo_example_11)/ros2_control/carlikebot.ros2_control.xacro" />
+  <xacro:include filename="$(find ros2_control_demo_example_7)/ros2_control/r6bot.ros2_control.xacro" />
   <xacro:carlikebot prefix="$(arg prefix)" />
-  <xacro:carlikebot_ros2_control
-    name="CarlikeBot" prefix="$(arg prefix)" />
+  <xacro:r6bot_description />
+  <xacro:carlikebot_ros2_control name="CarlikeBot" prefix="$(arg prefix)" />
+  <xacro:r6bot_ros2_control name="r6bot" />
+  <joint name="robots_joint" type="fixed">
+    <parent link="$(arg prefix)chassis_link" />
+    <child link="base_link" />
+    <origin xyz="0.2 0 0.03" rpy="0 0 0"/>
+  </joint>
 </robot>

File: my_workspace/src/ros2_control_demos/example_7/description/urdf/r6bot.urdf.xacro (robot description, xacro)
@@ -4,6 +4,5 @@
   <xacro:include filename="$(find ros2_control_demo_description)/r6bot/urdf/r6bot_description.urdf.xacro"/>
   <!-- create link fixed to the "world" -->
-  <link name="world"/>
-  <xacro:r6bot_description/>
+  <!--<link name="world"/> UNCOMMENT IF YOU WANT TO USE JUST MANIPULATOR WITHOUT CAR-->
   <!-- Import r6bot ros2_control description -->
   <xacro:include filename="$(find ros2_control_demo_example_7)/ros2_control/r6bot.ros2_control.xacro" />

File: my_workspace/src/ros2_control_demos/ros2_control_demo_description/r6bot/urdf/inc/create_link.xacro (robot description, xacro)
@@ -6,10 +6,11 @@
         rpy_offset
         mesh_package
-        mesh_name">
+        mesh_name
+        mesh_scale:= '1 1 1'">
     <link name="${link_name}">
       <visual>
         <origin xyz="${xyz_offset}" rpy="${rpy_offset}"/>
         <geometry>
-          <mesh filename="package://${mesh_package}/meshes/visual/${mesh_name}.dae"/>
+          <mesh filename="package://${mesh_package}/meshes/visual/${mesh_name}.dae" scale="${mesh_scale}"/>
         </geometry>
       </visual>
@@ -17,5 +18,5 @@
         <origin xyz="${xyz_offset}" rpy="${rpy_offset}"/>
         <geometry>
-          <mesh filename="package://${mesh_package}/meshes/collision/${mesh_name}.stl"/>
+          <mesh filename="package://${mesh_package}/meshes/collision/${mesh_name}.stl" scale="${mesh_scale}"/>
         </geometry>
       </collision>

File: my_workspace/src/ros2_control_demos/ros2_control_demo_description/r6bot/urdf/r6bot_description.urdf.xacro (robot description, xacro)
@@ -10,46 +10,53 @@
       mesh_package="ros2_control_demo_description/r6bot"
       mesh_name="link_0"
+      mesh_scale="0.2 0.2 0.2"
   />
   <xacro:create_link
       link_name="link_1"
-      xyz_offset="0 0 -0.182"
+      xyz_offset="0 0 ${-0.182 * 0.2}"
       rpy_offset="0 0 0"
       mesh_package="ros2_control_demo_description/r6bot"
       mesh_name="link_1"
+      mesh_scale="0.2 0.2 0.2"
   />
   <xacro:create_link
       link_name="link_2"
-      xyz_offset="0 0 -0.168"
+      xyz_offset="0 0 ${-0.168 * 0.2}"
       rpy_offset="0 0 0"
       mesh_package="ros2_control_demo_description/r6bot"
       mesh_name="link_2"
+      mesh_scale="0.2 0.2 0.2"
   />
   <xacro:create_link
       link_name="link_3"
-      xyz_offset="0 0 -0.144"
+      xyz_offset="0 0 ${-0.144 * 0.2}"
       rpy_offset="0 0 0"
       mesh_package="ros2_control_demo_description/r6bot"
       mesh_name="link_3"
+      mesh_scale="0.2 0.2 0.2"
   />
   <xacro:create_link
       link_name="link_4"
-      xyz_offset="0 0 0.077"
+      xyz_offset="0 0 ${0.077 * 0.2}"
       rpy_offset="0 0 0"
       mesh_package="ros2_control_demo_description/r6bot"
       mesh_name="link_4"
+      mesh_scale="0.2 0.2 0.2"
   />
   <xacro:create_link
       link_name="link_5"
-      xyz_offset="0 0 0.113"
+      xyz_offset="0 0 ${0.113 * 0.2}"
       rpy_offset="0 0 0"
       mesh_package="ros2_control_demo_description/r6bot"
       mesh_name="link_5"
+      mesh_scale="0.2 0.2 0.2"
   />
   <xacro:create_link
       link_name="link_6"
-      xyz_offset="0 0 0.086"
+      xyz_offset="0 0 ${0.086 * 0.2}"
       rpy_offset="0 0 0"
       mesh_package="ros2_control_demo_description/r6bot"
       mesh_name="link_6"
+      mesh_scale="0.2 0.2 0.2"
   />
   <link name="ft_frame"/>
@@ -57,5 +64,6 @@
   <!-- base_joint fixes base_link to the environment -->
   <joint name="base_joint" type="fixed">
-    <parent link="world"/>
+    <!--<parent link="world"/> USE THIS IF YOU WANT TO USE JUST MANIPULATOR WITHOUT CAR-->
+    <parent link="car_chassis_link"/>
     <child link="base_link"/>
     <origin xyz="0 0 0" rpy="0 0 0"/>
@@ -66,5 +74,5 @@
     <parent link="base_link"/>
     <child link="link_1"/>
-    <origin xyz="0 0 0.244" rpy="0 0 0"/>
+    <origin xyz="0 0 ${0.244 * 0.2}" rpy="0 0 0"/>
     <axis xyz="0 0 1"/>
     <limit effort="1000.0" lower="${-pi}" upper="${pi}" velocity="2.5"/>
@@ -73,5 +81,5 @@
     <parent link="link_1"/>
     <child link="link_2"/>
-    <origin xyz="-0.27 0 0.0" rpy="${-pi/2} -${pi/2} ${pi/2}"/>
+    <origin xyz="${-0.27 * 0.2} 0 0.0" rpy="${-pi/2} -${pi/2} ${pi/2}"/>
     <axis xyz="0 0 1"/>
     <limit effort="1000.0" lower="${-pi}" upper="${pi}" velocity="2.5"/>
@@ -80,5 +88,5 @@
     <parent link="link_2"/>
     <child link="link_3"/>
-    <origin xyz="0.686 0 -0.27" rpy="0 ${pi} ${pi+pi/2}"/>
+    <origin xyz="${0.686 * 0.2} 0 ${-0.27 * 0.2}" rpy="0 ${pi} ${pi+pi/2}"/>
     <axis xyz="0 0 1"/>
     <limit effort="1000.0" lower="${-pi}" upper="${pi}" velocity="2.5"/>
@@ -87,5 +95,5 @@
     <parent link="link_3"/>
     <child link="link_4"/>
-    <origin xyz="0.519 0 0" rpy="0 ${pi} ${pi}"/>
+    <origin xyz="${0.519 * 0.2} 0 0" rpy="0 ${pi} ${pi}"/>
     <axis xyz="0 0 1"/>
     <limit effort="1000.0" lower="${-pi}" upper="${pi}" velocity="2.5"/>
@@ -94,5 +102,5 @@
     <parent link="link_4"/>
     <child link="link_5"/>
-    <origin xyz="0.0 0 0.188" rpy="${pi/2} ${pi} ${pi/2}"/>
+    <origin xyz="0.0 0 ${0.188 * 0.2}" rpy="${pi/2} ${pi} ${pi/2}"/>
     <axis xyz="0 0 1"/>
     <limit effort="1000.0" lower="${-pi}" upper="${pi}" velocity="2.5"/>
@@ -101,5 +109,5 @@
     <parent link="link_5"/>
     <child link="link_6"/>
-    <origin xyz="0.0 0 0.246" rpy="0 ${-pi/2} 0"/>
+    <origin xyz="0.0 0 ${0.246 * 0.2}" rpy="0 ${-pi/2} 0"/>
     <axis xyz="0 0 1"/>
     <limit effort="1000.0" lower="${-pi}" upper="${pi}" velocity="2.5"/>
@@ -108,10 +116,10 @@
     <parent link="link_6"/>
     <child link="ft_frame"/>
-    <origin xyz="0 0 0.086" rpy="0 0 0"/>
+    <origin xyz="0 0 ${0.086 * 0.2}" rpy="0 0 0"/>
   </joint>
   <joint name="joint-tool" type="fixed">
     <parent link="ft_frame"/>
     <child link="tool0"/>
-    <origin xyz="0 0 0.185" rpy="0 0 0"/>
+    <origin xyz="0 0 ${0.185 * 0.2}" rpy="0 0 0"/>
   </joint>
 </xacro:macro>
